File: hardware/Flunkerboy/eingangsteiler.kicad_sch (KiCad schematic)
At the start: 62 parts, among them J2 Conn_01x01_Socket, J3 Conn_01x01_Socket, J4 Conn_01x01_Socket, K1 AGQ200A4HZ, K2 AGQ200A4HZ, K3 AGQ200A4HZ, K4 AGQ200A4HZ, SW1 SW_SPST, U2 ADG734, U3 ADG734, U4 ADG1611, U5 ADG1611, U6 ADG1611, U7 ADG1611, U8 ADG1611

Commit message: add docs
Parts:
- removed C17, C18, C19, C20: 100n, Capacitor_SMD:C_0805_2012Metric, symbol Device:C
- removed J4: Conn_01x01_Socket, Connector:Banana_Cliff_FCR7350B_S16N-PC_Horizontal, symbol Connector:Conn_01x01_Socket
- removed K1, K2, K3, K4: AGQ200A4HZ, Relay_THT:Relay_DPDT_Omron_G6K-2P-Y, symbol Relay:Relay_DPDT
- removed R9: 0.012, Resistor_SMD:R_0805_2012Metric, symbol Device:R
- removed RV10: 100k, Resistor_SMD:R_0805_2012Metric, symbol Device:R_Potentiometer
- removed SW1: SW_SPST, symbol Switch:SW_SPST
- removed U2, U3: ADG734, Package_SO:TSSOP-20_4.4x6.5mm_P0.65mm, symbol Analog_Switch:ADG734
- added D11, D12, D13, D5: 1N4148, Diode_SMD:D_SOD-123, symbol Diode:1N4007
- added RL1, RL3, RL4, RL6: AGQ200A4HZ, Relay_THT:Relay_DPDT_Omron_G6K-2P-Y, symbol Relay:JW2
- RV41: footprint Resistor_SMD:R_0805_2012Metric -> Potentiometer_SMD:Potentiometer_Bourns_3224J_Horizontal
- U4, U5, U6, U7, U8: LCSC part (none) -> C377682
Connections:
- net A: now also RL6.6
- net B: now also RL6.3
- net D: now also RL1.3
- net GND: now also D11.2 (A), D12.2 (A), D13.2 (A), D5.2 (A), RL1.8, RL3.1, RL4.1, RL6.8
- net GNDA: now also RL1.2, RL6.4
- net S3a: now also D13.1 (K), RL3.8
- net S4b: now also D12.1 (K), RL4.8
- net S5a: now also D5.1 (K), RL1.1
- net S5c: now also D11.1 (K), RL6.1
- net at U5.10 (D3), U6.10 (D3), U7.15 (D2)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: now also RL4.5, RL6.7
- net at D1.2 (A), D2.1 (K), U4.10 (D3)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: now also RL4.4
- net at R1.1, U5.11 (S3), U8.11 (S3): now also RL3.2
- net at U4.15 (D2), U5.2 (D1), U6.2 (D1)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: now also RL1.4
- net at R2.2, R3.1, U4.11 (S3)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: now also RL4.6
- net at F1.2: now also RL4.3
- net at RV41.2: now also RL6.2
- new net: RL3.4, RL6.5
- new net: RL3.3, RL4.2
- no-connect marks 0 -> 7
Other:
- note removed: "20A!"
- moved on the sheet: C10, C11, C2, C3, C4, C5, C6, C7, C8, C9, U4E, U5E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
